File: ProjectAurora/LED-Controller.kicad_sch (KiCad schematic)
At the start: 18 parts, among them IC1 IS31FL3237-QFLS4-TR

Commit message: Starting Layout
Parts:
- C13, C14, C15: footprint (none) -> Capacitor_SMD:C_0603_1608Metric
- D1, D10, D11, D12, D2, D3, D4, D5, D6, D7, D8, D9: footprint (none) -> LED:XL-1615RGBC-YG; symbol Device:LED_RGBA -> XINGLIGHT XL-1615RGBC-YG:XL-1615RGBC-YG
- IC1: footprint IS31FL3237QFLS4TR -> IS31LF3237:IS31FL3237QFLS4TR
- R11, R12: footprint (none) -> Resistor_SMD:R_0603_1608Metric
Connections:
- net +3V3: now also D1.1 (A), D10.1 (A), D11.1 (A), D12.1 (A), D2.1 (A), D3.1 (A), D4.1 (A), D5.1 (A), D6.1 (A), D7.1 (A), D8.1 (A), D9.1 (A); no longer D1.4 (A), D10.4 (A), D11.4 (A), D12.4 (A), D2.4 (A), D3.4 (A), D4.4 (A), D5.4 (A), D6.4 (A), D7.4 (A), D8.4 (A), D9.4 (A)
- net OUT1: now also D6.4 (RK); no longer D1.1 (RK)
- net OUT10: now also D3.4 (RK); no longer D4.1 (RK)
- net OUT11: now also D3.3 (GK); no longer D4.2 (GK)
- net OUT12: now also D3.2 (BK); no longer D4.3 (BK)
- net OUT13: now also D2.4 (RK); no longer D5.1 (RK)
- net OUT14: now also D2.3 (GK); no longer D5.2 (GK)
- net OUT15: now also D2.2 (BK); no longer D5.3 (BK)
- net OUT16: now also D1.4 (RK); no longer D6.1 (RK)
- net OUT17: now also D1.3 (GK); no longer D6.2 (GK)
- net OUT18: now also D1.2 (BK); no longer D6.3 (BK)
- net OUT19: now also D7.4 (RK); no longer D7.1 (RK)
- net OUT2: now also D6.3 (GK); no longer D1.2 (GK)
- net OUT20: now also D7.3 (GK); no longer D7.2 (GK)
- net OUT21: now also D7.2 (BK); no longer D7.3 (BK)
- net OUT22: now also D8.4 (RK); no longer D8.1 (RK)
- net OUT23: now also D8.3 (GK); no longer D8.2 (GK)
- net OUT24: now also D8.2 (BK); no longer D8.3 (BK)
- net OUT25: now also D9.4 (RK); no longer D9.1 (RK)
- net OUT26: now also D9.3 (GK); no longer D9.2 (GK)
- net OUT27: now also D9.2 (BK); no longer D9.3 (BK)
- net OUT28: now also D10.4 (RK); no longer D10.1 (RK)
- net OUT29: now also D10.3 (GK); no longer D10.2 (GK)
- net OUT3: now also D6.2 (BK); no longer D1.3 (BK)
- net OUT30: now also D10.2 (BK); no longer D10.3 (BK)
- net OUT31: now also D11.4 (RK); no longer D11.1 (RK)
- net OUT32: now also D11.3 (GK); no longer D11.2 (GK)
- net OUT33: now also D11.2 (BK); no longer D11.3 (BK)
- net OUT34: now also D12.4 (RK); no longer D12.1 (RK)
- net OUT35: now also D12.3 (GK); no longer D12.2 (GK)
- net OUT36: now also D12.2 (BK); no longer D12.3 (BK)
- net OUT4: now also D5.4 (RK); no longer D2.1 (RK)
- net OUT5: now also D5.3 (GK); no longer D2.2 (GK)
- net OUT6: now also D5.2 (BK); no longer D2.3 (BK)
- net OUT7: now also D4.4 (RK); no longer D3.1 (RK)
- net OUT8: now also D4.3 (GK); no longer D3.2 (GK)
- net OUT9: now also D4.2 (BK); no longer D3.3 (BK)

Commit message: Prototype Board Layout Done
Parts:
- added B1, B10, B11, B12, B2, B3, B4, B5, B6, B8, B9, G1, G10, G11, G12, G2, G3, G4, G5, G6, G7, G8, G9, RED1, RED10, RED11, RED12, RED2, RED3, RED4, RED5, RED6, RED7, RED8, RED9: TestPoint, TestPoint:TestPoint_Pad_1.0x1.0mm, symbol Connector:TestPoint
- added B7: `, TestPoint:TestPoint_Pad_1.0x1.0mm, symbol Connector:TestPoint
- renumbered D9 to D10, D8 to D11, D7 to D12, D12 to D7, D11 to D8, D10 to D9
Connections:
- net OUT1: now also RED6.1
- net OUT10: now also RED3.1
- net OUT11: now also G3.1
- net OUT12: now also B3.1
- net OUT13: now also RED2.1
- net OUT14: now also G2.1
- net OUT15: now also B2.1
- net OUT16: now also RED1.1
- net OUT17: now also G1.1
- net OUT18: now also B1.1
- net OUT19: now also RED12.1
- net OUT2: now also G6.1
- net OUT20: now also G12.1
- net OUT21: now also B12.1
- net OUT22: now also RED11.1
- net OUT23: now also G11.1
- net OUT24: now also B11.1
- net OUT25: now also RED10.1
- net OUT26: now also G10.1
- net OUT27: now also B10.1
- net OUT28: now also RED9.1
- net OUT29: now also G9.1
- net OUT3: now also B6.1
- net OUT30: now also B9.1
- net OUT31: now also RED8.1
- net OUT32: now also G8.1
- net OUT33: now also B8.1
- net OUT34: now also RED7.1
- net OUT35: now also G7.1
- net OUT36: now also B7.1
- net OUT4: now also RED5.1
- net OUT5: now also G5.1
- net OUT6: now also B5.1
- net OUT7: now also RED4.1
- net OUT8: now also G4.1
- net OUT9: now also B4.1

Commit message: Prototype Board Ready for Ordering
Parts:
- renumbered D2 to D1, D11 to D10, D12 to D11, D1 to D12, D3 to D2, D4 to D3, D5 to D4, D6 to D5, D7 to D6, D8 to D7, D9 to D8, D10 to D9
Changed lines of the file:
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@@
 		(dnp no)
 		(fields_autoplaced yes)
-		(property "Reference" "D7"
+		(property "Reference" "D6"
 			(at 231.14 139.7 0)
 			(effects
@@
 			(project "ProjectAurora"
 				(path "/3ca855de-33e1-4742-b952-4e80ee0f08b6/48cdbbd7-34d6-4c6d-b523-5eee0bb171ae"
-					(reference "D7")
+					(reference "D6")
 					(unit 1)
 				)
@@
 		(dnp no)
 		(fields_autoplaced yes)
-		(property "Reference" "D11"
+		(property "Reference" "D10"
 			(at 231.14 44.45 0)
 			(effects
@@
 			(project "ProjectAurora"
 				(path "/3ca855de-33e1-4742-b952-4e80ee0f08b6/48cdbbd7-34d6-4c6d-b523-5eee0bb171ae"
-					(reference "D11")
+					(reference "D10")
 					(unit 1)
 				)
@@
 		(dnp no)
 		(fields_autoplaced yes)
-		(property "Reference" "D3"
+		(property "Reference" "D2"
 			(at 200.66 67.31 0)
 			(effects
@@
 			(project "ProjectAurora"
 				(path "/3ca855de-33e1-4742-b952-4e80ee0f08b6/48cdbbd7-34d6-4c6d-b523-5eee0bb171ae"
-					(reference "D3")
+					(reference "D2")
 					(unit 1)
 				)
@@
 		(dnp no)
 		(fields_autoplaced yes)
-		(property "Reference" "D8"
+		(property "Reference" "D7"
 			(at 231.14 115.57 0)
 			(effects
@@
 			(project "ProjectAurora"
 				(path "/3ca855de-33e1-4742-b952-4e80ee0f08b6/48cdbbd7-34d6-4c6d-b523-5eee0bb171ae"
-					(reference "D8")
+					(reference "D7")
 					(unit 1)
 				)
@@
 		(dnp no)
 		(fields_autoplaced yes)
-		(property "Reference" "D4"
+		(property "Reference" "D3"
 			(at 200.66 91.44 0)
 			(effects
@@
 			(project "ProjectAurora"
 				(path "/3ca855de-33e1-4742-b952-4e80ee0f08b6/48cdbbd7-34d6-4c6d-b523-5eee0bb171ae"
-					(reference "D4")
+					(reference "D3")
 					(unit 1)
 				)
@@
 		(dnp no)
 		(fields_autoplaced yes)
-		(property "Reference" "D12"
+		(property "Reference" "D11"
 			(at 231.14 20.32 0)
 			(effects
@@
 			(project "ProjectAurora"
 				(path "/3ca855de-33e1-4742-b952-4e80ee0f08b6/48cdbbd7-34d6-4c6d-b523-5eee0bb171ae"
-					(reference "D12")
+					(reference "D11")
 					(unit 1)
 				)
@@
 		(dnp no)
 		(fields_autoplaced yes)
-		(property "Reference" "D6"
+		(property "Reference" "D5"
 			(at 200.66 139.7 0)
 			(effects
@@
 			(project "ProjectAurora"
 				(path "/3ca855de-33e1-4742-b952-4e80ee0f08b6/48cdbbd7-34d6-4c6d-b523-5eee0bb171ae"
-					(reference "D6")
+					(reference "D5")
 					(unit 1)
 				)
@@
 		(dnp no)
 		(fields_autoplaced yes)
-		(property "Reference" "D10"
+		(property "Reference" "D9"
 			(at 231.14 67.31 0)
 			(effects
@@
 			(project "ProjectAurora"
 				(path "/3ca855de-33e1-4742-b952-4e80ee0f08b6/48cdbbd7-34d6-4c6d-b523-5eee0bb171ae"
-					(reference "D10")
+					(reference "D9")
 					(unit 1)
 				)
@@
 		(dnp no)
 		(fields_autoplaced yes)
-		(property "Reference" "D1"
+		(property "Reference" "D12"
 			(at 200.66 19.05 0)
 			(effects
@@
 			(project "ProjectAurora"
 				(path "/3ca855de-33e1-4742-b952-4e80ee0f08b6/48cdbbd7-34d6-4c6d-b523-5eee0bb171ae"
-					(reference "D1")
+					(reference "D12")
 					(unit 1)
 				)
@@
 		(dnp no)
 		(fields_autoplaced yes)
-		(property "Reference" "D9"
+		(property "Reference" "D8"
 			(at 231.14 91.44 0)
 			(effects
@@
 			(project "ProjectAurora"
 				(path "/3ca855de-33e1-4742-b952-4e80ee0f08b6/48cdbbd7-34d6-4c6d-b523-5eee0bb171ae"
-					(reference "D9")
+					(reference "D8")
 					(unit 1)
 				)
@@
 		(dnp no)
 		(fields_autoplaced yes)
-		(property "Reference" "D2"
+		(property "Reference" "D1"
 			(at 200.66 43.18 0)
 			(effects
@@
 			(project "ProjectAurora"
 				(path "/3ca855de-33e1-4742-b952-4e80ee0f08b6/48cdbbd7-34d6-4c6d-b523-5eee0bb171ae"
-					(reference "D2")
+					(reference "D1")
 					(unit 1)
 				)
@@
 		(dnp no)
 		(fields_autoplaced yes)
-		(property "Reference" "D5"
+		(property "Reference" "D4"
 			(at 200.66 115.57 0)
 			(effects
@@
 			(project "ProjectAurora"
 				(path "/3ca855de-33e1-4742-b952-4e80ee0f08b6/48cdbbd7-34d6-4c6d-b523-5eee0bb171ae"
-					(reference "D5")
+					(reference "D4")
 					(unit 1)
 				)
